Commit message: Fixed links

File: src/motoman_robot/motoman_description/robots/motomini/motomini_basic.urdf.xacro (robot description, xacro)
@@ -21,13 +21,4 @@
                                        + link_3_u_volume  + link_4_r_volume
                                        + link_5_b_volume  + link_6_t_volume}" />
-    <!-- Add macro -->
-    <xacro:macro name="add_world" params="*origin">
-      <link name="world"/>
-      <joint name="world" type="fixed">
-        <insert_block name="origin"/>
-        <parent link="world"/>
-        <child link="base_link"/>
-      </joint>
-    </xacro:macro>
     <!-- link list -->
     <!--
@@ -65,4 +56,13 @@
     <link name="tool0"/>
     <!-- end of link list -->
+    <!-- Add macro -->
+    <xacro:macro name="add_world" params="*origin">
+      <link name="world"/>
+      <joint name="world" type="fixed">
+        <insert_block name="origin"/>
+        <parent link="world"/>
+        <child link="base_link"/>
+      </joint>
+    </xacro:macro>
     <!-- joint list -->
     <xacro:joint_v0 joint_name="${prefix}joint_1_s"

File: src/motoman_robot/motoman_description/robots/motomini/motomini_with_gripper_kinectv2.urdf.xacro (robot description, xacro)
@@ -7,5 +7,5 @@
   <xacro:include filename="$(find motoman_description)/urdf/sensor/kinect.gazebo.xacro"/>
   <xacro:include filename="$(find motoman_description)/urdf/tool/gripper.urdf.xacro" />
-  <xacro:include filename="$(find motoman_description)/urdf/mount/cammount.urdf.xacro" />
+  <xacro:include filename="$(find motoman_description)/urdf/mount/cammount.urdf.xacro"/>
   <!-- Include gazebo grasp_fix plugin -->
   <xacro:if value="$(arg load_grasp_fix)">
@@ -21,27 +21,8 @@
   <xacro:mymount name="mymount">
   </xacro:mymount>
-  <!-- <xacro:mymount name="mount_link"/> -->
-  <!-- <link name="mount_link_x"/>
-  Joint -->
-  <!-- <joint name="joint_mount_x" type="fixed">
-    <origin xyz="0.4 0.4 0" rpy="0 0.0 0"/>
-    <parent link="world"/>
-    <child link="mount_link"/>
-    <dynamics damping="0.5" friction="0.0"/>
-  </joint> -->
-  <!-- <xacro:simple_jp_trans_v0 name="transmission_1_s"
-                              joint_name="joint_mount" actuator_name="motor_1_j"
-                              reduction="300"/> -->
-  <!-- <joint name="joint_rgb_kinect2" type="fixed"> -->
-    <!-- <origin rpy="${M_PI/2} ${M_PI} ${M_PI/2}"/> -->
-    <!-- <parent link="kinect2_link"/> -->
-    <!-- <child link="kinect2_rgb_optical_frame"/> -->
-  <!-- </joint> -->
-  <!-- Gazebo -->
-  <!-- <xacro:kinect_gazebo name="kinect2"/> -->
-  <!-- <xacro:sensor_d435 parent="mount_link_1">
-      <origin xyz="0.1 0 0.10" rpy="0 0.5 0"/>
-   </xacro:sensor_d435> -->
-  <!-- <link name="kinect2_rgb_optical_frame"/> -->
+  <!-- add Kinect V2 -->
+  <!-- Link -->
+  <!-- <xacro:kinect2_link_box_v0 name="kinect2_link"/>
+  <link name="kinect2_rgb_optical_frame"/> -->
   <!-- Joint -->
   <!-- <joint name="joint_kinect2" type="fixed">
@@ -49,6 +30,6 @@
     <parent link="base_link"/>
     <child link="kinect2_link"/>
-  </joint>
-  <joint name="joint_rgb_kinect2" type="fixed">
+  </joint> -->
+  <!-- <joint name="joint_rgb_kinect2" type="fixed">
     <origin rpy="${M_PI/2} ${M_PI} ${M_PI/2}"/>
     <parent link="kinect2_link"/>
@@ -56,8 +37,4 @@
   </joint> -->
   <!-- Gazebo -->
-  <!-- <xacro:gazebo_d435/> -->
-  <!-- <xacro:sensor_d435 parent="${prefix}base_link">
-  </xacro:sensor_d435> -->
-  <!-- add Kinect V2 -->
-  <!-- Link -->
+  <!-- <xacro:kinect_gazebo name="kinect2"/> -->
 </robot>

File: src/motoman_robot/motoman_description/urdf/mount/cammount.urdf.xacro (robot description, xacro)
@@ -4,13 +4,43 @@
 <xacro:include filename="$(find motoman_description)/urdf/sensor/_d435.gazebo.xacro"/>
 <xacro:macro name="mymount" params="name">
+    <link name='mount_base_link'>
+      <inertial>
+      <origin xyz="0 0 0.025" rpy="0 0 0"/>
+        <mass value ="0.5"/>
+        <inertia
+          ixx = "0.001"
+          ixy="0"
+          ixz="0"
+          iyy="0.001"
+          iyz="0"
+          izz="0.001"
+        />
+        <pose frame=''>0 0 0 0 -0 0</pose>
+      </inertial>
+      <visual name='visual'>
+      <origin xyz="0 0 0.025"/>
+        <geometry>
+          <box size = "0.06 0.06 0.05"/>
+        </geometry>
+        <material name="Gazebo/Black"/>
+      </visual>
+      <collision name='collision'>
+      <origin xyz="0 0 0.025"/>
+        <geometry>
+          <box size = "0.06 0.06 0.05"/>
+        </geometry>
+        <material name="Gazebo/Black"/>
+      </collision>
+      <gazebo>
+        <material>Gazebo/Blue</material>
+        <!-- <material>Gazebo/Black</material> -->
+      </gazebo>
+    </link>
     <joint name="mountjoint" type="fixed" >
-      <axis xyz="0 0 1" />
-      <!-- <insert_block name="origin" /> -->
-      <origin xyz="0.07 0.10 0.28"/>
-      <parent link="base_link" />
-      <child link="mount_link" />
-      <limit upper="-1000000" lower="100000" effort="-1" velocity="10"/>
-    </joint>
-    <link name='mount_link'>
+      <origin xyz="0 0.2 0"/>
+      <parent link="world" />
+      <child link="mount_base_link" />
+    </joint>
+    <link name='mount_bod'>
       <inertial>
         <mass value ="0.521791"/>
@@ -34,5 +64,5 @@
         </geometry>
         <material name="Gazebo/Black"/>
-        <gazebo reference="mount_link">
+        <gazebo reference="mount_bod">
           <material>Gazebo/Black</material>
         </gazebo>
@@ -95,4 +125,25 @@
       </collision>
     </link>
+    <joint name='bod_base_link' type='revolute'>
+      <parent link="mount_base_link"/>
+      <child link="mount_bod"/>
+      <!-- <pose frame=''>0 0 0 0 -0 0</pose> -->
+      <origin xyz="0 0 0.3811" rpy="0 0 0" />
+      <axis xyz="0 0 1" />
+      <limit upper="1" lower="-1" effort="1" velocity="1"/>
+      <dynamics spring_reference="0" spring_stiffness="0" damping="0"/>
+      <physics>
+        <ode>
+          <limit>
+            <cfm>0</cfm>
+            <erp>0.2</erp>
+          </limit>
+          <suspension>
+            <cfm>0</cfm>
+            <erp>0.2</erp>
+          </suspension>
+        </ode>
+      </physics>
+    </joint>
     <link name='mount_link_1'>
       <inertial>
@@ -110,5 +161,5 @@
       <pose frame=''>0.033479 0.001202 -0.001243 0 -0 1.2e-05</pose>
       <visual name='visual'>
-      <origin xyz="0.033479 0.001202 0.2243"/>
+      <!-- <origin xyz="0.033479 0.001202 0.2243"/> -->
         <pose frame=''>0 0 0 0 -0 0</pose>
         <geometry>
@@ -123,5 +174,5 @@
       </visual>
       <collision name='collision'>
-      <origin xyz="0.033479 0.001202 0.2243"/>
+      <!-- <origin xyz="0.033479 0.001202 0.2243"/> -->
         <laser_retro>0</laser_retro>
         <max_contacts>10</max_contacts>
@@ -177,10 +228,11 @@
       </collision>
     </link>
-    <joint name='link_JOINT_1' type='fixed'>
-      <parent link="mount_link"/>
+    <joint name='link_JOINT_1' type='revolute'>
+      <parent link="mount_bod"/>
       <child link="mount_link_1"/>
+      <origin xyz="0.033479 0.001202 0.2543"/>
       <!-- <pose frame=''>0 0 0 0 -0 0</pose> -->
       <axis xyz="0 1 0" />
-      <limit upper="-1" lower="1" effort="-1" velocity="-1"/>
+      <limit upper="0" lower="-0.61" effort="1" velocity="1"/>
       <dynamics spring_reference="0" spring_stiffness="0" damping="0"/>
       <!-- <axis>
@@ -207,6 +259,26 @@
       </physics>
     </joint>
+    <transmission name="tran1">
+    <type>transmission_interface/SimpleTransmission</type>
+    <joint name="bod_base_link">
+      <hardwareInterface>hardware_interface/EffortJointInterface</hardwareInterface>
+    </joint>
+    <actuator name="motor1">
+      <hardwareInterface>hardware_interface/EffortJointInterface</hardwareInterface>
+      <mechanicalReduction>1</mechanicalReduction>
+    </actuator>
+  </transmission>
+    <!-- <transmission name="tran2">
+    <type>transmission_interface/SimpleTransmission</type>
+    <joint name="link_JOINT_1">
+      <hardwareInterface>hardware_interface/EffortJointInterface</hardwareInterface>
+    </joint>
+    <actuator name="motor1">
+      <hardwareInterface>hardware_interface/EffortJointInterface</hardwareInterface>
+      <mechanicalReduction>1</mechanicalReduction>
+    </actuator>
+  </transmission> -->
   <xacro:sensor_d435 parent="mount_link_1">
-      <origin xyz="0.05 0 0.2043" rpy="0 0.95 0"/>
+      <origin xyz="0.01376 0 0" rpy="0 0.6 0"/>
    </xacro:sensor_d435>
 </xacro:macro>
