Commit message: moveit_added_demo

File: src/motoman_robot/motoman_description/robots/motomini/motomini_with_gripper_kinectv2.urdf.xacro (robot description, xacro)
@@ -17,5 +17,5 @@
   <!-- add gripper -->
   <xacro:gripper name="gripper" parent="tool0">
-    <origin xyz="0 0 0.0035" rpy="0 0 0" />
+    <origin xyz="0 0 0.025" rpy="0 0 0" />
   </xacro:gripper>
   <xacro:mymount name="mymount">

File: src/motoman_robot/motoman_description/urdf/motomini/body.urdf.xacro (robot description, xacro)
@@ -59,7 +59,7 @@
 	<origin xyz="${origin_xyz}" rpy="${origin_rpy}"/>
         <mass value="${mass}"/>
-        <inertia ixx="${(mass*((width/2)*(width/2)+(height/2)*(height/2)))/3}" ixy="0" ixz="0"
-				 iyy="${(mass*((depth/2)*(depth/2)+(height/2)*(height/2)))/3}" iyz="0"
-				 izz="${(mass*((depth/2)*(depth/2)+(width/2)*(width/2)))/3}" />
+        <inertia ixx="${(mass*((width/2)*(width/2)+(height/2)*(height/2)))/12}" ixy="0" ixz="0"
+				 iyy="${(mass*((depth/2)*(depth/2)+(height/2)*(height/2)))/12}" iyz="0"
+				 izz="${(mass*((depth/2)*(depth/2)+(width/2)*(width/2)))/12}" />
       </inertial>
     </link>
@@ -74,4 +74,5 @@
       <axis xyz="${axis_xyz}" />
       <limit lower="${llimit}" upper="${ulimit}" effort="${elimit}" velocity="${vlimit}"/>
+      <dynamics damping="5" friction="0.1"/>
     </joint>
   </xacro:macro>

File: src/motoman_robot/motoman_description/urdf/mount/cammount.urdf.xacro (robot description, xacro)
@@ -262,8 +262,8 @@
     <type>transmission_interface/SimpleTransmission</type>
     <joint name="bod_base_link">
-      <hardwareInterface>hardware_interface/EffortJointInterface</hardwareInterface>
+      <hardwareInterface>hardware_interface/PositionJointInterface</hardwareInterface>
     </joint>
     <actuator name="motor1">
-      <hardwareInterface>hardware_interface/EffortJointInterface</hardwareInterface>
+      <hardwareInterface>hardware_interface/PositionJointInterface</hardwareInterface>
       <mechanicalReduction>1</mechanicalReduction>
     </actuator>
@@ -272,8 +272,8 @@
     <type>transmission_interface/SimpleTransmission</type>
     <joint name="link_JOINT_1">
-      <hardwareInterface>hardware_interface/EffortJointInterface</hardwareInterface>
+      <hardwareInterface>hardware_interface/PositionJointInterface</hardwareInterface>
     </joint>
     <actuator name="motor1">
-      <hardwareInterface>hardware_interface/EffortJointInterface</hardwareInterface>
+      <hardwareInterface>hardware_interface/PositionJointInterface</hardwareInterface>
       <mechanicalReduction>1</mechanicalReduction>
     </actuator>

File: src/motoman_robot/motoman_description/urdf/tool/gripper.gazebo.xacro (robot description, xacro)
@@ -1,7 +1,4 @@
 <?xml version="1.0"?>
-<robot xmlns:sensor="http://playerstage.sourceforge.net/gazebo/xmlschema/#sensor"
-       xmlns:controller="http://playerstage.sourceforge.net/gazebo/xmlschema/#controller"
-       xmlns:interface="http://playerstage.sourceforge.net/gazebo/xmlschema/#interface"
-       xmlns:xacro="http://ros.org/wiki/xacro">
+<robot xmlns:xacro="http://ros.org/wiki/xacro">
   <xacro:macro name="gripper_gazebo" params="name">
     <gazebo reference="${name}_palm_link">
@@ -10,5 +7,5 @@
       <selfCollide>false</selfCollide>
     </gazebo>
-    <gazebo reference="${name}_finger_l_link">
+    <gazebo reference="${name}_finger_link_r">
       <material>Gazebo/Black</material>
       <turnGravityOff>false</turnGravityOff>
@@ -16,7 +13,19 @@
       <mu1>1.0</mu1>
       <mu2>1.0</mu2>
+      <minDepth>0.001</minDepth>
       <maxContacts>100</maxContacts>
+      <sensor name="finger_r_contact" type="contact">
+        <always_on>1</always_on>
+        <contact>
+          <collision>gripper_finger_link_r_collision</collision>
+        </contact>
+        <plugin name="gripper_bumper_r" filename="libgazebo_ros_bumper.so">
+          <alwaysOn>true</alwaysOn>
+          <bumperTopicName>gripper_finger_link_r_collision</bumperTopicName>
+          <frameName>gripper_finger_r_link</frameName>
+        </plugin>
+      </sensor>
     </gazebo>
-    <gazebo reference="${name}_finger_r_link">
+    <gazebo reference="${name}_finger_link_l">
       <material>Gazebo/Black</material>
       <turnGravityOff>false</turnGravityOff>
@@ -24,5 +33,17 @@
       <mu1>1.0</mu1>
       <mu2>1.0</mu2>
+      <minDepth>0.001</minDepth>
       <maxContacts>100</maxContacts>
+      <sensor name="finger_l_contact" type="contact">
+        <always_on>1</always_on>
+        <contact>
+          <collision>gripper_finger_link_l_collision</collision>
+        </contact>
+        <plugin name="gripper_bumper_l" filename="libgazebo_ros_bumper.so">
+          <alwaysOn>true</alwaysOn>
+          <bumperTopicName>gripper_finger_link_l_collision</bumperTopicName>
+          <frameName>gripper_finger_l_link</frameName>
+        </plugin>
+      </sensor>
     </gazebo>
   </xacro:macro>

File: src/motoman_robot/motoman_description/urdf/tool/gripper.transmission.xacro (robot description, xacro)
@@ -8,9 +8,9 @@
       <type>transmission_interface/SimpleTransmission</type>
       <actuator name="${name}_finger_l_motor">
-        <hardwareInterface>hardware_interface/EffortJointInterface</hardwareInterface>
+        <hardwareInterface>hardware_interface/PositionJointInterface</hardwareInterface>
         <mechanicalReduction>1</mechanicalReduction>
       </actuator>
       <joint name="${name}_finger_joint_l">
-        <hardwareInterface>hardware_interface/EffortJointInterface</hardwareInterface>
+        <hardwareInterface>hardware_interface/PositionJointInterface</hardwareInterface>
       </joint>
     </transmission>
@@ -18,9 +18,9 @@
       <type>transmission_interface/SimpleTransmission</type>
       <actuator name="${name}_finger_r_motor">
-        <hardwareInterface>hardware_interface/EffortJointInterface</hardwareInterface>
+        <hardwareInterface>hardware_interface/PositionJointInterface</hardwareInterface>
         <mechanicalReduction>1</mechanicalReduction>
       </actuator>
       <joint name="${name}_finger_joint_r">
-        <hardwareInterface>hardware_interface/EffortJointInterface</hardwareInterface>
+        <hardwareInterface>hardware_interface/PositionJointInterface</hardwareInterface>
       </joint>
     </transmission>

Commit message: corrected gripper and damping

File: src/motoman_robot/motoman_description/robots/motomini/motomini_with_gripper_kinectv2.urdf.xacro (robot description, xacro)
@@ -17,5 +17,5 @@
   <!-- add gripper -->
   <xacro:gripper name="gripper" parent="tool0">
-    <origin xyz="0 0 0.0035" rpy="0 0 0" />
+    <origin xyz="0 0 0.026" rpy="0 0 0" />
   </xacro:gripper>
   <xacro:mymount name="mymount">

File: src/motoman_robot/motoman_description/urdf/motomini/body.urdf.xacro (robot description, xacro)
@@ -59,7 +59,7 @@
 	<origin xyz="${origin_xyz}" rpy="${origin_rpy}"/>
         <mass value="${mass}"/>
-        <inertia ixx="${(mass*((width/2)*(width/2)+(height/2)*(height/2)))/3}" ixy="0" ixz="0"
-				 iyy="${(mass*((depth/2)*(depth/2)+(height/2)*(height/2)))/3}" iyz="0"
-				 izz="${(mass*((depth/2)*(depth/2)+(width/2)*(width/2)))/3}" />
+        <inertia ixx="${(mass*((width/2)*(width/2)+(height/2)*(height/2)))/12}" ixy="0" ixz="0"
+				 iyy="${(mass*((depth/2)*(depth/2)+(height/2)*(height/2)))/12}" iyz="0"
+				 izz="${(mass*((depth/2)*(depth/2)+(width/2)*(width/2)))/12}" />
       </inertial>
     </link>
@@ -73,4 +73,5 @@
       <origin xyz="${origin_xyz}" rpy="${origin_rpy}" />
       <axis xyz="${axis_xyz}" />
+      <dynamics damping="1"/>
       <limit lower="${llimit}" upper="${ulimit}" effort="${elimit}" velocity="${vlimit}"/>
     </joint>

File: src/motoman_robot/motoman_description/urdf/tool/gripper.gazebo.xacro (robot description, xacro)
@@ -10,5 +10,5 @@
       <selfCollide>false</selfCollide>
     </gazebo>
-    <gazebo reference="${name}_finger_l_link">
+    <gazebo reference="${name}_finger_link_l">
       <material>Gazebo/Black</material>
       <turnGravityOff>false</turnGravityOff>
@@ -18,5 +18,5 @@
       <maxContacts>100</maxContacts>
     </gazebo>
-    <gazebo reference="${name}_finger_r_link">
+    <gazebo reference="${name}_finger_link_r">
       <material>Gazebo/Black</material>
       <turnGravityOff>false</turnGravityOff>

Commit message: before moveitgripper

File: src/motoman_robot/motoman_description/robots/motomini/motomini_with_gripper_kinectv2.urdf.xacro (robot description, xacro)
@@ -17,5 +17,5 @@
   <!-- add gripper -->
   <xacro:gripper name="gripper" parent="tool0">
-    <origin xyz="0 0 0.026" rpy="0 0 0" />
+    <origin xyz="0 0 0.020" rpy="0 0 0" />
   </xacro:gripper>
   <xacro:mymount name="mymount">

Commit message: works-mostly

File: src/motoman_robot/motoman_description/robots/motomini/motomini_with_gripper_kinectv2.urdf.xacro (robot description, xacro)
@@ -2,5 +2,5 @@
 <robot name="motoman_motomini" xmlns:xacro="http://ros.org/wiki/xacro">
   <!-- Arguments -->
-  <xacro:arg name="load_grasp_fix" default="false"/>
+  <xacro:arg name="load_grasp_fix" default="true"/>
   <!-- Include Sensors -->
   <xacro:include filename="$(find motoman_description)/urdf/sensor/kinect.urdf.xacro"/>

File: src/motoman_robot/motoman_description/urdf/tool/gripper.gazebo.xacro (robot description, xacro)
@@ -14,7 +14,7 @@
       <turnGravityOff>false</turnGravityOff>
       <selfCollide>true</selfCollide>
-      <mu1>3.0</mu1>
-      <mu2>3.0</mu2>
-      <!-- <maxContacts>100</maxContacts> -->
+      <mu1>1.0</mu1>
+      <mu2>1.0</mu2>
+      <maxContacts>100</maxContacts>
     </gazebo>
     <gazebo reference="${name}_finger_link_r">
@@ -22,7 +22,7 @@
       <turnGravityOff>false</turnGravityOff>
       <selfCollide>true</selfCollide>
-      <mu1>3.0</mu1>
-      <mu2>3.0</mu2>
-      <!-- <maxContacts>100</maxContacts> -->
+      <mu1>1.0</mu1>
+      <mu2>1.0</mu2>
+      <maxContacts>100</maxContacts>
     </gazebo>
   </xacro:macro>

File: src/motoman_robot/motoman_description/urdf/tool/gripper.urdf.xacro (robot description, xacro)
@@ -41,6 +41,6 @@
       <axis xyz="0 -1 0" />
       <dynamics damping="1.0" friction="1.0" />
-      <limit effort="100" velocity="10" lower="0" upper="${finger_joint}"/>
-      <safety_controller k_position="20" k_velocity="25" soft_lower_limit="${threshold}" soft_upper_limit="${finger_joint_soft}" />
+      <limit effort="200" velocity="0.1" lower="0" upper="${finger_joint}"/>
+      <!-- <safety_controller k_position="20" k_velocity="25" soft_lower_limit="${threshold}" soft_upper_limit="${finger_joint_soft}" /> -->
     </joint>
     <link name="${name}_finger_link_l">
@@ -48,5 +48,5 @@
         <origin xyz="0 -0.001 0" rpy="0 0 0" />
         <mass value="0.01"/>
-        <inertia ixx="0.01" ixy="0" ixz="0" iyy="0.01" iyz="0" izz="0.01" />
+        <inertia ixx="0.001" ixy="0" ixz="0" iyy="0.001" iyz="0" izz="0.001" />
       </inertial>
       <visual>
@@ -69,8 +69,8 @@
       <parent link="${name}_palm_link"/>
       <child link="${name}_finger_link_r"/>
-      <axis xyz="0 -1 0" />
+      <axis xyz="0 1 0" />
       <dynamics damping="1.0" friction="1.0" />
-      <limit effort="100" velocity="10" lower="0" upper="${finger_joint}"/>
-      <safety_controller k_position="20" k_velocity="25" soft_lower_limit="${threshold}" soft_upper_limit="${finger_joint_soft}" />
+      <limit effort="200" velocity="0.1" upper="0" lower="-${finger_joint}"/>
+      <!-- <safety_controller k_position="20" k_velocity="25" soft_uper_limit="-${threshold}" soft_lower_limit="-${finger_joint_soft}" /> -->
     </joint>
     <link name="${name}_finger_link_r">
@@ -78,5 +78,5 @@
         <origin xyz="0.000 -0.001 0" rpy="0 0 0" />
         <mass value="0.01"/>
-        <inertia ixx="0.01" ixy="0" ixz="0" iyy="0.01" iyz="0" izz="0.01" />
+        <inertia ixx="0.001" ixy="0" ixz="0" iyy="0.001" iyz="0" izz="0.001" />
       </inertial>
       <visual>
