Commit message: Fixed transforms and mounts

File: src/motoman_robot/motoman_description/urdf/mount/cammount.urdf.xacro (robot description, xacro)
@@ -234,5 +234,5 @@
       <!-- <pose frame=''>0 0 0 0 -0 0</pose> -->
       <axis xyz="0 1 0" />
-      <limit upper="0" lower="-0.61" effort="1" velocity="1"/>
+      <limit upper="0.61" lower="-0.61" effort="1" velocity="1"/>
       <dynamics spring_reference="0" spring_stiffness="0" damping="0"/>
       <!-- <axis>
@@ -269,5 +269,5 @@
     </actuator>
   </transmission>
-    <!-- <transmission name="tran2">
+    <transmission name="tran2">
     <type>transmission_interface/SimpleTransmission</type>
     <joint name="link_JOINT_1">
@@ -278,5 +278,5 @@
       <mechanicalReduction>1</mechanicalReduction>
     </actuator>
-  </transmission> -->
+  </transmission>
   <xacro:sensor_d435 parent="mount_link_1">
       <origin xyz="0.01376 0 0" rpy="0 0.6 0"/>

Commit message: rebuilt with description

File: src/motoman_robot/motoman_description/urdf/mount/cammount.urdf.xacro (robot description, xacro)
@@ -38,5 +38,5 @@
     </link>
     <joint name="mountjoint" type="fixed" >
-      <origin xyz="0 0.2 0"/>
+      <origin xyz="0 0.3 0"/>
       <parent link="world" />
       <child link="mount_base_link" />
@@ -61,5 +61,5 @@
       <visual name='visual'>
         <geometry>
-          <box size="0.042409 0.050234 0.682253"/>
+          <box size="0.042409 0.050234 0.502253"/>
         </geometry>
         <material name="Gazebo/Black"/>
@@ -76,5 +76,5 @@
         <pose frame=''>0 0 0 0 -0 0</pose>
         <geometry>
-          <box size="0.042409 0.050234 0.682253"/>
+          <box size="0.042409 0.050234 0.502253"/>
         </geometry>
         <surface>
@@ -129,5 +129,5 @@
       <child link="mount_bod"/>
       <!-- <pose frame=''>0 0 0 0 -0 0</pose> -->
-      <origin xyz="0 0 0.3811" rpy="0 0 0" />
+      <origin xyz="0 0 0.2911" rpy="0 0 0" />
       <axis xyz="0 0 1" />
       <limit upper="1" lower="-1" effort="1" velocity="1"/>
@@ -231,8 +231,8 @@
       <parent link="mount_bod"/>
       <child link="mount_link_1"/>
-      <origin xyz="0.033479 0.001202 0.2543"/>
+      <origin xyz="0.033479 0.001202 0.1643"/>
       <!-- <pose frame=''>0 0 0 0 -0 0</pose> -->
       <axis xyz="0 1 0" />
-      <limit upper="0.61" lower="-0.61" effort="1" velocity="1"/>
+      <limit upper="0.61" lower="-0.61" effort="0.5" velocity="0.5"/>
       <dynamics spring_reference="0" spring_stiffness="0" damping="0"/>
       <!-- <axis>
