Commit message: mastercommit

File: src/motoman_robot/motoman_description/urdf/tool/gripper.gazebo.xacro (robot description, xacro)
@@ -14,7 +14,7 @@
       <turnGravityOff>false</turnGravityOff>
       <selfCollide>true</selfCollide>
-      <mu1>1.0</mu1>
-      <mu2>1.0</mu2>
-      <maxContacts>100</maxContacts>
+      <mu1>3.0</mu1>
+      <mu2>3.0</mu2>
+      <!-- <maxContacts>100</maxContacts> -->
     </gazebo>
     <gazebo reference="${name}_finger_link_r">
@@ -22,7 +22,7 @@
       <turnGravityOff>false</turnGravityOff>
       <selfCollide>true</selfCollide>
-      <mu1>1.0</mu1>
-      <mu2>1.0</mu2>
-      <maxContacts>100</maxContacts>
+      <mu1>3.0</mu1>
+      <mu2>3.0</mu2>
+      <!-- <maxContacts>100</maxContacts> -->
     </gazebo>
   </xacro:macro>

File: src/motoman_robot/motoman_description/urdf/tool/gripper.urdf.xacro (robot description, xacro)
@@ -41,5 +41,5 @@
       <axis xyz="0 -1 0" />
       <dynamics damping="1.0" friction="1.0" />
-      <limit effort="2" velocity="0.1" lower="0" upper="${finger_joint}"/>
+      <limit effort="100" velocity="10" lower="0" upper="${finger_joint}"/>
       <safety_controller k_position="20" k_velocity="25" soft_lower_limit="${threshold}" soft_upper_limit="${finger_joint_soft}" />
     </joint>
@@ -71,5 +71,5 @@
       <axis xyz="0 -1 0" />
       <dynamics damping="1.0" friction="1.0" />
-      <limit effort="2" velocity="0.1" lower="0" upper="${finger_joint}"/>
+      <limit effort="100" velocity="10" lower="0" upper="${finger_joint}"/>
       <safety_controller k_position="20" k_velocity="25" soft_lower_limit="${threshold}" soft_upper_limit="${finger_joint_soft}" />
     </joint>
