Commit message: cleaned

File: src/motoman_robot/motoman_description/urdf/tool/gripper.urdf.xacro (robot description, xacro)
@@ -48,5 +48,5 @@
         <origin xyz="0 -0.001 0" rpy="0 0 0" />
         <mass value="0.01"/>
-        <inertia ixx="0.001" ixy="0" ixz="0" iyy="0.001" iyz="0" izz="0.001" />
+        <inertia ixx="0.000173" ixy="0" ixz="0" iyy="0.000165" iyz="-0.000018" izz="0.000039" />
       </inertial>
       <visual>
@@ -78,5 +78,5 @@
         <origin xyz="0.000 -0.001 0" rpy="0 0 0" />
         <mass value="0.01"/>
-        <inertia ixx="0.001" ixy="0" ixz="0" iyy="0.001" iyz="0" izz="0.001" />
+        <inertia ixx="0.000173" ixy="0" ixz="0" iyy="0.000165" iyz="-0.000018" izz="0.000039" />
       </inertial>
       <visual>
